Commit message: Wheel position correction URDF file

File: urdf/diff_robot.urdf (robot description, URDF)
Before this commit: robot diff_robot, 5 links, 4 joints
Joints:
- joint left_wheel_joint: origin xyz=0 0.3125 0.0 rpy=0 0 0 -> xyz=0 0.3 0.0 rpy=0 0 0
- joint right_wheel_joint: origin xyz=0 -0.3125 0.0 rpy=0 0 0 -> xyz=0 -0.3 0.0 rpy=0 0 0
